Commit message: Feat: Add support for testing parallel simulation environments

File: diffusion_policy/env_runner/robotiq_ur10e/ur10e_robotiq.urdf (robot description, URDF)
Before this commit: robot ur10e_robotiq, 23 links, 22 joints
Links:
- link eef: geometry visual sphere radius=0.005
Joints:
- joint left_inner_finger_joint: mimic joint=left_inner_knuckle_joint multiplier=1.0 offset=0.0 -> joint=left_outer_knuckle_joint multiplier=1.0 offset=0.0
- joint right_inner_finger_joint: mimic joint=right_inner_knuckle_joint multiplier=1.0 offset=0.0 -> joint=right_outer_knuckle_joint multiplier=1.0 offset=0.0
